File: KiCad PCB/Fingerprint_doorbell.kicad_sch (KiCad schematic)
At the start: 13 parts, among them J1 Conn_01x06_Pin, J2 Screw_Terminal_01x02, J3 Screw_Terminal_01x02, J4 Conn_01x03_Pin, J5 Conn_01x06_Pin, J6 Conn_01x07_Pin, U1 ESP32-S3_ZERO, U2 LTV-817S

Commit message: foodprint fixed
Parts:
- U1: footprint esp32kicadlibrary:MODULE_ESP32-S3_ZERO -> lib:MODULE_ESP32-S3_ZERO
Changed lines of the file:
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@@
 			)
 		)
-		(property "Footprint" "esp32kicadlibrary:MODULE_ESP32-S3_ZERO"
+		(property "Footprint" "lib:MODULE_ESP32-S3_ZERO"
 			(at 55.118 101.092 0)
 			(effects
